File: Hardware/design/design.sch (KiCad schematic (older format))
At the start: 67 parts, among them SW1 Alps_SRBV, SW10 Alps_SRBV, SW11 SW_Push, SW12 SW_Push, SW13 SW_Push, SW14 SW_Push, SW16 SW_Push, SW17 SW_Push, SW18 SW_Push, SW19 SW_Push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

Commit message: added mounting holes, rounded edges and silkscreen
Parts:
- added H1, H2, H3, H4: MountingHole, MountingHole:MountingHole_4mm, symbol Mechanical:MountingHole
Connections:
- net labels removed: ROW6
Changed lines of the file:
@@
 $EndComp
 Text Label 3650 7200 0    50   ~ 0
-ROW6
+ROW5
 Text Label 2800 7200 0    50   ~ 0
-ROW6
-Text Label 2800 5200 0    50   ~ 0
 ROW5
 Text Label 3650 5200 0    50   ~ 0
-ROW5
+ROW4
+Text Label 2800 5200 0    50   ~ 0
+ROW4
+$Comp
+L Mechanical:MountingHole H2
+U 1 1 61514673
+P 10300 6150
+F 0 "H2" H 10400 6196 50  0000 L CNN
+F 1 "MountingHole" H 10400 6105 50  0000 L CNN
+F 2 "MountingHole:MountingHole_4mm" H 10300 6150 50  0001 C CNN
+F 3 "~" H 10300 6150 50  0001 C CNN
+	1    10300 6150
+	1    0    0    -1
+$EndComp
+$Comp
+L Mechanical:MountingHole H4
+U 1 1 61515309
+P 10600 6150
+F 0 "H4" H 10700 6196 50  0000 L CNN
+F 1 "MountingHole" H 10700 6105 50  0000 L CNN
+F 2 "MountingHole:MountingHole_4mm" H 10600 6150 50  0001 C CNN
+F 3 "~" H 10600 6150 50  0001 C CNN
+	1    10600 6150
+	1    0    0    -1
+$EndComp
+$Comp
+L Mechanical:MountingHole H1
+U 1 1 6151D16C
+P 10300 5900
+F 0 "H1" H 10400 5946 50  0000 L CNN
+F 1 "MountingHole" H 10400 5855 50  0000 L CNN
+F 2 "MountingHole:MountingHole_4mm" H 10300 5900 50  0001 C CNN
+F 3 "~" H 10300 5900 50  0001 C CNN
+	1    10300 5900
+	1    0    0    -1
+$EndComp
+$Comp
+L Mechanical:MountingHole H3
+U 1 1 6151D172
+P 10600 5900
+F 0 "H3" H 10700 5946 50  0000 L CNN
+F 1 "MountingHole" H 10700 5855 50  0000 L CNN
+F 2 "MountingHole:MountingHole_4mm" H 10600 5900 50  0001 C CNN
+F 3 "~" H 10600 5900 50  0001 C CNN
+	1    10600 5900
+	1    0    0    -1
+$EndComp
 $EndSCHEMATC

Commit message: library management
Connections:
- no-connect marks 0 -> 8
Other:
- note added: "2 octave matrix"
- note added: "MIDI control change potentiometers"
- note added: "MIDI_keyboard V1"
- note added: "Scanning process pseudocode:\n\nInit(){\n for row in rows{\n setmode(row, INPUT_PULLUP);\n }\n for col in cols{\n setmode(col, OUTPUT);\n write(col,1);\n } \n}\ndef scan_row(row){\n for col in cols{\n write(col, 0);\n if(read(row) == 0){\n //button at (row,col) is pressed\n }\n write(col, 1);\n }\n}"
- note added: "left and right octave select"
- note added: "mounting holes"
- note removed: "Scanning process pseudocode:\n\nInit(){\nfor row in rows{\nsetmode(row, INPUT_PULLUP);\n}\nfor col in cols{\nsetmode(col, OUTPUT);\nwrite(col,1);\n} \n}\ndef scan_row(row){\nfor col in cols{\nwrite(col, 0);\nif(read(row) == 0){\n//button at (row,col) is pressed\n}\nwrite(col, 1);\n}\n}"
- moved on the sheet: H1, H2
Changed lines of the file:
@@
 Text Label 1550 1850 0    50   ~ 0
 VCC
-Wire Wire Line
-	5200 3000 5500 3000
 Text Label 5250 3000 0    50   ~ 0
 VCC
@@
 Text Label 1050 2300 0    50   ~ 0
 GND
-Wire Wire Line
-	5200 2800 5500 2800
 Text Label 5250 2800 0    50   ~ 0
 GND
@@
 RAW
 Text Notes 4800 2150 0    50   ~ 0
-Scanning process pseudocode:\n\nInit(){\nfor row in rows{\nsetmode(row, INPUT_PULLUP);\n}\nfor col in cols{\nsetmode(col, OUTPUT);\nwrite(col,1);\n} \n}\ndef scan_row(row){\nfor col in cols{\nwrite(col, 0);\nif(read(row) == 0){\n//button at (row,col) is pressed\n}\nwrite(col, 1);\n}\n}
+Scanning process pseudocode:\n\nInit(){\n  for row in rows{\n    setmode(row, INPUT_PULLUP);\n  }\n  for col in cols{\n    setmode(col, OUTPUT);\n    write(col,1);\n  } \n}\ndef scan_row(row){\n  for col in cols{\n    write(col, 0);\n    if(read(row) == 0){\n      //button at (row,col) is pressed\n    }\n    write(col, 1);\n  }\n}
 $Comp
 L pspice:DIODE D12
@@
 L Mechanical:MountingHole H2
 U 1 1 61514673
-P 10300 6150
-F 0 "H2" H 10400 6196 50  0000 L CNN
-F 1 "MountingHole" H 10400 6105 50  0000 L CNN
-F 2 "MountingHole:MountingHole_4mm" H 10300 6150 50  0001 C CNN
-F 3 "~" H 10300 6150 50  0001 C CNN
-	1    10300 6150
+P 9800 6150
+F 0 "H2" H 9900 6196 50  0000 L CNN
+F 1 "MountingHole" H 9900 6105 50  0000 L CNN
+F 2 "MountingHole:MountingHole_4mm" H 9800 6150 50  0001 C CNN
+F 3 "~" H 9800 6150 50  0001 C CNN
+	1    9800 6150
 	1    0    0    -1
 $EndComp
@@
 L Mechanical:MountingHole H1
 U 1 1 6151D16C
-P 10300 5900
-F 0 "H1" H 10400 5946 50  0000 L CNN
-F 1 "MountingHole" H 10400 5855 50  0000 L CNN
-F 2 "MountingHole:MountingHole_4mm" H 10300 5900 50  0001 C CNN
-F 3 "~" H 10300 5900 50  0001 C CNN
-	1    10300 5900
+P 9800 5900
+F 0 "H1" H 9900 5946 50  0000 L CNN
+F 1 "MountingHole" H 9900 5855 50  0000 L CNN
+F 2 "MountingHole:MountingHole_4mm" H 9800 5900 50  0001 C CNN
+F 3 "~" H 9800 5900 50  0001 C CNN
+	1    9800 5900
 	1    0    0    -1
 $EndComp
@@
 	1    0    0    -1
 $EndComp
+Text Notes 7900 750  0    118  ~ 24
+2 octave matrix
+Text Notes 700  1500 0    118  ~ 24
+MIDI control change potentiometers
+Text Notes 9750 5650 0    118  ~ 24
+mounting holes
+Text Notes 1550 4500 0    118  ~ 24
+left and right octave select
+NoConn ~ 5500 2700
+NoConn ~ 5500 2900
+NoConn ~ 3450 2700
+NoConn ~ 3450 2800
+NoConn ~ 3650 5000
+NoConn ~ 3650 5100
+NoConn ~ 3650 7300
+NoConn ~ 3650 7400
+Wire Wire Line
+	5200 2800 5500 2800
+Wire Wire Line
+	5200 3000 5500 3000
+$Comp
+L power:PWR_FLAG #FLG0101
+U 1 1 615FDBC4
+P 5500 3000
+F 0 "#FLG0101" H 5500 3075 50  0001 C CNN
+F 1 "PWR_FLAG" V 5500 3128 50  0000 L CNN
+F 2 "" H 5500 3000 50  0001 C CNN
+F 3 "~" H 5500 3000 50  0001 C CNN
+	1    5500 3000
+	0    1    1    0
+$EndComp
+$Comp
+L power:PWR_FLAG #FLG0102
+U 1 1 615FF50C
+P 5500 2800
+F 0 "#FLG0102" H 5500 2875 50  0001 C CNN
+F 1 "PWR_FLAG" V 5500 2928 50  0000 L CNN
+F 2 "" H 5500 2800 50  0001 C CNN
+F 3 "~" H 5500 2800 50  0001 C CNN
+	1    5500 2800
+	0    1    1    0
+$EndComp
+Text Notes 7050 6950 0    157  ~ 31
+MIDI_keyboard V1
 $EndSCHEMATC

Commit message: switched COL0 and COL2 positions on the rotary switches
Changed lines of the file:
@@
 Text Label 5250 2700 0    50   ~ 0
 RAW
-Text Notes 4800 2150 0    50   ~ 0
-Scanning process pseudocode:\n\nInit(){\n  for row in rows{\n    setmode(row, INPUT_PULLUP);\n  }\n  for col in cols{\n    setmode(col, OUTPUT);\n    write(col,1);\n  } \n}\ndef scan_row(row){\n  for col in cols{\n    write(col, 0);\n    if(read(row) == 0){\n      //button at (row,col) is pressed\n    }\n    write(col, 1);\n  }\n}
 $Comp
 L pspice:DIODE D12
@@
 	5100 5850 5100 6550
 Wire Wire Line
-	2500 5850 2500 6550
-Wire Wire Line
 	1800 5850 1800 6550
 Wire Wire Line
 	1300 5850 1300 6550
-Text Label 1300 6150 0    50   ~ 0
-COL0
 Text Label 1800 6150 0    50   ~ 0
 COL1
-Text Label 2500 6150 0    50   ~ 0
-COL2
 Text Label 850  6150 0    50   ~ 0
 COL3
@@
 Text Notes 7050 6950 0    157  ~ 31
 MIDI_keyboard V1
+Text Notes 4800 2150 0    50   ~ 0
+Scanning process pseudocode:\n\nInit(){\n  for row in rows{\n    setmode(row, INPUT_PULLUP);\n  }\n  for col in cols{\n    setmode(col, OUTPUT);\n    write(col,1);\n  } \n}\ndef scan_row(row){\n  for col in cols{\n    write(col, 0);\n    if(read(row) == 0){\n      //button at (row,col) is pressed\n    }\n    write(col, 1);\n  }\n}
+Wire Wire Line
+	2500 5850 2500 6550
+Text Label 2500 6150 0    50   ~ 0
+COL0
+Text Label 1300 6150 0    50   ~ 0
+COL2
 $EndSCHEMATC
