File: Hardware/design/design.kicad_pcb (KiCad board)
At the start: 2 copper layers, 285.8 x 85.1 mm, 71 parts, among them SW1 Alps_SRBV, SW10 Alps_SRBV, SW11 SW_Push, SW12 SW_Push, SW13 SW_Push, SW14 SW_Push, SW16 SW_Push, SW17 SW_Push, SW18 SW_Push, SW19 SW_Push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

Commit message: commiting before better routing branch
Routing:
- net /COL1: track 399.6 -> 398.6 mm
- net /GND: vias 0 -> 47
- net (no net): vias 0 -> 1
- added copper zone on B.Cu, net /GND
- added copper zone on F.Cu, net /GND
Changed lines of the file:
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@@
     (thickness 1.6)
     (drawings 21)
-    (tracks 634)
+    (tracks 680)
     (zones 0)
     (modules 71)
@@
     (pad_to_mask_clearance 0)
     (aux_axis_origin 0 0)
+    (grid_origin 43.15 86.75)
     (visible_elements 7FFFFFFF)
     (pcbplotparams
@@
     (effects (font (size 4 4) (thickness 0.35)))
   )
+  (via (at 158.325 79.95) (size 0.8) (drill 0.4) (layers F.Cu B.Cu) (net 2))
+  (via (at 46.8 87.55) (size 0.8) (drill 0.4) (layers F.Cu B.Cu) (net 2))
+  (via (at 43.925 90.675) (size 0.8) (drill 0.4) (layers F.Cu B.Cu) (net 2))
+  (via (at 35.875 90.575) (size 0.8) (drill 0.4) (layers F.Cu B.Cu) (net 2))
+  (via (at 31.45 88.825) (size 0.8) (drill 0.4) (layers F.Cu B.Cu) (net 2))
+  (via (at 28.5 88.425) (size 0.8) (drill 0.4) (layers F.Cu B.Cu) (net 2))
+  (via (at 22.725 88.525) (size 0.8) (drill 0.4) (layers F.Cu B.Cu) (net 2))
+  (via (at 66.725 101.75) (size 0.8) (drill 0.4) (layers F.Cu B.Cu) (net 2))
+  (via (at 78.525 112.575) (size 0.8) (drill 0.4) (layers F.Cu B.Cu) (net 0))
+  (via (at 126.85 101.85) (size 0.8) (drill 0.4) (layers F.Cu B.Cu) (net 2))
+  (via (at 131.6 112.775) (size 0.8) (drill 0.4) (layers F.Cu B.Cu) (net 2))
+  (via (at 179.5 118.175) (size 0.8) (drill 0.4) (layers F.Cu B.Cu) (net 2))
+  (via (at 142.525 105.55) (size 0.8) (drill 0.4) (layers F.Cu B.Cu) (net 2))
+  (via (at 119.625 107.375) (size 0.8) (drill 0.4) (layers F.Cu B.Cu) (net 2))
+  (via (at 180.075 124.525) (size 0.8) (drill 0.4) (layers F.Cu B.Cu) (net 2))
+  (via (at 182.325 112.925) (size 0.8) (drill 0.4) (layers F.Cu B.Cu) (net 2))
   (segment (start 101.6 67.91) (end 100.374999 69.135001) (width 0.25) (layer F.Cu) (net 1))
   (segment (start 118.199998 67.91) (end 101.6 67.91) (width 0.25) (layer F.Cu) (net 1))
@@
   (segment (start 16.880001 70.424999) (end 65.985001 70.424999) (width 0.25) (layer B.Cu) (net 2))
   (segment (start 15.755 71.55) (end 16.880001 70.424999) (width 0.25) (layer B.Cu) (net 2))
+  (via (at 222.8 75.1) (size 0.8) (drill 0.4) (layers F.Cu B.Cu) (net 2))
+  (via (at 213.275 81.325) (size 0.8) (drill 0.4) (layers F.Cu B.Cu) (net 2))
+  (via (at 207.15 100.325) (size 0.8) (drill 0.4) (layers F.Cu B.Cu) (net 2))
+  (via (at 195.225 115.8) (size 0.8) (drill 0.4) (layers F.Cu B.Cu) (net 2))
+  (via (at 259.475 57.225) (size 0.8) (drill 0.4) (layers F.Cu B.Cu) (net 2))
+  (via (at 136.95 124) (size 0.8) (drill 0.4) (layers F.Cu B.Cu) (net 2))
+  (via (at 116.225 124.9) (size 0.8) (drill 0.4) (layers F.Cu B.Cu) (net 2))
+  (via (at 104.5 122.975) (size 0.8) (drill 0.4) (layers F.Cu B.Cu) (net 2))
+  (via (at 80.475 115.8) (size 0.8) (drill 0.4) (layers F.Cu B.Cu) (net 2))
+  (via (at 70.125 110.525) (size 0.8) (drill 0.4) (layers F.Cu B.Cu) (net 2))
+  (via (at 67.95 112.875) (size 0.8) (drill 0.4) (layers F.Cu B.Cu) (net 2))
+  (via (at 71.425 120.6) (size 0.8) (drill 0.4) (layers F.Cu B.Cu) (net 2))
+  (via (at 80.05 102.5) (size 0.8) (drill 0.4) (layers F.Cu B.Cu) (net 2))
+  (via (at 166.1 97.025) (size 0.8) (drill 0.4) (layers F.Cu B.Cu) (net 2))
+  (via (at 57.7 105.175) (size 0.8) (drill 0.4) (layers F.Cu B.Cu) (net 2))
+  (via (at 229.925 61.925) (size 0.8) (drill 0.4) (layers F.Cu B.Cu) (net 2))
+  (via (at 229.825 64.35) (size 0.8) (drill 0.4) (layers F.Cu B.Cu) (net 2))
+  (via (at 229.95 67) (size 0.8) (drill 0.4) (layers F.Cu B.Cu) (net 2))
+  (via (at 252.95 61.9) (size 0.8) (drill 0.4) (layers F.Cu B.Cu) (net 2))
+  (via (at 201 61.825) (size 0.8) (drill 0.4) (layers F.Cu B.Cu) (net 2))
+  (via (at 177.8 61.7) (size 0.8) (drill 0.4) (layers F.Cu B.Cu) (net 2))
+  (via (at 177.8 64.45) (size 0.8) (drill 0.4) (layers F.Cu B.Cu) (net 2))
+  (via (at 177.775 66.7) (size 0.8) (drill 0.4) (layers F.Cu B.Cu) (net 2))
+  (via (at 189.225 71.25) (size 0.8) (drill 0.4) (layers F.Cu B.Cu) (net 2))
+  (via (at 49.75 95.15) (size 0.8) (drill 0.4) (layers F.Cu B.Cu) (net 2))
+  (via (at 40.75 96.525) (size 0.8) (drill 0.4) (layers F.Cu B.Cu) (net 2))
+  (via (at 23.775 57.95) (size 0.8) (drill 0.4) (layers F.Cu B.Cu) (net 2))
+  (via (at 21.15 57.95) (size 0.8) (drill 0.4) (layers F.Cu B.Cu) (net 2))
+  (via (at 26.4 57.975) (size 0.8) (drill 0.4) (layers F.Cu B.Cu) (net 2))
+  (via (at 34.925 57.925) (size 0.8) (drill 0.4) (layers F.Cu B.Cu) (net 2))
+  (via (at 32.425 57.925) (size 0.8) (drill 0.4) (layers F.Cu B.Cu) (net 2))
+  (via (at 29.75 58) (size 0.8) (drill 0.4) (layers F.Cu B.Cu) (net 2))
   (segment (start 59.2 74.71) (end 64.774999 69.135001) (width 0.25) (layer F.Cu) (net 3))
   (segment (start 48.375 74.71) (end 59.2 74.71) (width 0.25) (layer F.Cu) (net 3))
@@
   (via (at 202.641501 77.491501) (size 0.8) (drill 0.4) (layers F.Cu B.Cu) (net 26))
   (segment (start 203.94 76.193002) (end 202.641501 77.491501) (width 0.25) (layer F.Cu) (net 26))
-  (segment (start 198.715 77.51) (end 202.623002 77.51) (width 0.25) (layer B.Cu) (net 26))
-  (segment (start 182.425 93.8) (end 198.715 77.51) (width 0.25) (layer B.Cu) (net 26))
-  (segment (start 202.623002 77.51) (end 202.641501 77.491501) (width 0.25) (layer B.Cu) (net 26))
-  (segment (start 182.425 95.525) (end 182.425 93.8) (width 0.25) (layer B.Cu) (net 26))
   (segment (start 41.525 109.69) (end 52.48 109.69) (width 0.25) (layer B.Cu) (net 27))
   (segment (start 52.48 109.69) (end 55.355 109.69) (width 0.25) (layer B.Cu) (net 27))
@@
   (segment (start 187.946004 93.26) (end 205.897003 75.309001) (width 0.25) (layer F.Cu) (net 25))
   (segment (start 162.775 93.26) (end 187.946004 93.26) (width 0.25) (layer F.Cu) (net 25))
+  (segment (start 200.458499 77.491501) (end 182.425 95.525) (width 0.25) (layer B.Cu) (net 26))
+  (segment (start 202.641501 77.491501) (end 200.458499 77.491501) (width 0.25) (layer B.Cu) (net 26))
   (segment (start 236.15001 96.81999) (end 234.95 98.02) (width 0.25) (layer F.Cu) (net 27))
   (segment (start 236.15001 94.60682) (end 236.15001 96.81999) (width 0.25) (layer F.Cu) (net 27))
@@
   (segment (start 276.975 114.27) (end 275.575 115.67) (width 0.25) (layer F.Cu) (net 54))
   (segment (start 282.575 114.27) (end 276.975 114.27) (width 0.25) (layer F.Cu) (net 54))
+  (zone (net 2) (net_name /GND) (layer F.Cu) (hatch edge 0.508)
+    (connect_pads (clearance 0.508))
+    (min_thickness 0.254)
+    (fill yes (arc_segments 32) (thermal_gap 0.508) (thermal_bridge_width 0.508))
+    (polygon
+      (pts
+        (xy 298.6 31.975) (xy 298.4 142.8) (xy -13.925 143.175) (xy -12.8 28.6)
+      )
+    )
+  )
+  (zone (net 2) (net_name /GND) (layer B.Cu) (hatch edge 0.508)
+    (connect_pads (clearance 0.508))
+    (min_thickness 0.254)
+    (fill yes (arc_segments 32) (thermal_gap 0.508) (thermal_bridge_width 0.508))
+    (polygon
+      (pts
+        (xy 214.5 34.15) (xy 297.625 33.5) (xy 298.175 141.125) (xy -12.775 142.45) (xy -11.55 31.95)
+      )
+    )
+  )
 )

Commit message: routing has improved
Parts:
- turned D13 to 90 degrees
- turned D14 to 90 degrees
- turned D15 to 90 degrees
- turned D16 to 90 degrees
- turned D17 to 90 degrees
- turned D18 to 90 degrees
- turned D19 to 90 degrees
- turned D20 to 90 degrees
- turned D21 to 90 degrees
- turned D22 to 90 degrees
- turned D23 to 90 degrees
- turned D24 to 90 degrees
- turned D25 to 90 degrees
- turned D26 to 90 degrees
- turned D27 to 90 degrees
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Routing:
- net /COL5: track 439.2 -> 484.6 mm, vias 7 -> 4
- net /COL2: track 453.9 -> 420.4 mm, vias 16 -> 7
- net /COL3: track 447.2 -> 415.8 mm, vias 12 -> 7
- net /COL1: track 398.6 -> 423.7 mm, vias 13 -> 7
- net /ROW0: track 139.8 -> 121.2 mm
- net /COL4: track 426.4 -> 410.5 mm, vias 6 -> 4
- net /ROW2: track 263.0 -> 278.5 mm
- net /COL0: track 420.8 -> 431.4 mm, vias 10 -> 7
- net /ROW4: track 233.0 -> 239.4 mm, vias 2 -> 3
- net /ROW3: track 325.5 -> 330.8 mm
- net /ROW1: track 184.3 -> 189.2 mm
- net /ROW5: track 181.5 -> 185.4 mm
- net Net-(D13-Pad1): track 7.58 -> 10.5 mm
- net Net-(D28-Pad1): track 7.58 -> 10.1 mm
- net Net-(D33-Pad1): track 7.58 -> 9.80 mm
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- removed copper zone on F.Cu, net /GND

Commit message: board is now in production with JLCPCB
Routing:
- net /ROW5: track 185.4 -> 187.3 mm
- net /GND: vias 28 -> 50
- added copper zone on F.Cu, net /GND
